File: calciHATter/calciHATter.sch (KiCad schematic (older format))
At the start: 30 parts, among them J1 Screw_Terminal_01x02, J2 Jumper, J3 40HAT, U1 MAX31856, U2 CAT24C32

Commit message: PCB placement to include indicators and toggle switch
Parts:
- removed D2, D3, D4: LED, LED_SMD:LED_0603_1608Metric_Pad1.05x0.95mm_HandSolder, symbol Device:LED
- removed H1, H2, H3, H4: MountingHole_Pad, MountingHole:MountingHole_3.2mm_M3_Pad, symbol Mechanical:MountingHole_Pad
- removed J3: 40HAT, Connector_PinSocket_2.54mm:PinSocket_2x20_P2.54mm_Vertical, symbol calciHATter-rescue:OX40HAT-raspberrypi_hat
- removed R2, R3, R4: 1k, Resistor_SMD:R_0603_1608Metric_Pad1.05x0.95mm_HandSolder, symbol Device:R
- removed TP1, TP2, TP3, TP4, TP5, TP6: TestPoint, Connector_PinHeader_1.00mm:PinHeader_1x01_P1.00mm_Vertical, symbol Connector:TestPoint
- removed U2: CAT24C32, Package_SOIC:SOIC-8_3.9x4.9mm_P1.27mm, symbol calciHATter-rescue:CAT24C32-raspberrypi_hat
- added D1, D3, D4, D5, D6: GREEN, 0603, LED_SMD:LED_0603_1608Metric_Pad1.05x0.95mm_HandSolder, symbol Device:LED_Small
- added D2: RED, 0603, LED_SMD:LED_0603_1608Metric_Pad1.05x0.95mm_HandSolder, symbol Device:LED_Small
- added H1, H2, H3, H4: MountingHole, project_footprints:NPTH_3mm_ID, symbol Mechanical:MountingHole
- added J3: PI40HAT, Connector_PinSocket_2.54mm:PinSocket_2x20_P2.54mm_Vertical, symbol calciHATter:PI40HAT
- added J4: Conn_02x06_Odd_Even, Connector_PinHeader_2.54mm:PinHeader_2x06_P2.54mm_Vertical, symbol Connector_Generic:Conn_02x06_Odd_Even
- added R1, R2, R3, R4, R8, R9: 1k, 0603, Resistor_SMD:R_0603_1608Metric_Pad1.05x0.95mm_HandSolder, symbol Device:R_Small
- added R10: 10k, 0603, 1%, Resistor_SMD:R_0603_1608Metric_Pad1.05x0.95mm_HandSolder, symbol Device:R
- added R?: R, symbol Device:R
- added U2: CAT24C32, Package_SO:SOIC-8_3.9x4.9mm_P1.27mm, symbol calciHATter:CAT24C32
- added U3: CPC1125N, Package_SO:SOP-4_3.8x4.1mm_P2.54mm, symbol Relay_SolidState:ASSR-1218
Connections:
- net +3V3: now also J3.1 (P3V3), J3.17 (P3V3), J4.11 (Pin_11), U2.8 (VCC), U3.4; no longer C4.2, C5.2, U1.5 (AVDD), U1.8 (DVDD)
- net +5C: now also J3.2 (P5V), J3.4 (P5V)
- net FAULT: now also J3.36 (BCM16), J4.7 (Pin_7)
- net GND: now also C1.2, C2.1, D1.1 (K), D2.1 (K), D3.1 (K), D4.1 (K), D5.1 (K), D6.1 (K), J3.14 (GND), J3.20 (GND), J3.25 (GND), J3.30 (GND), J3.34 (GND), J3.39 (GND), J3.6 (GND), J3.9 (GND), R10.2, R?.1, U2.1 (A0), U2.2 (A1), U2.3 (A2), U2.4 (GND), U3.2; no longer C1.1, C2.2
- net HBEAT: now also J3.38 (BCM20), J4.9 (Pin_9)
- net ID_SC_EEPROM: now also J3.28 (BCM1), U2.5 (SDA)
- net ID_SD_EEPROM: now also J3.27 (BCM0), U2.6 (SCL)
- net MISO: now also J3.21 (BCM9), J4.3 (Pin_3)
- net MOSI: now also J3.19 (BCM10), J4.1 (Pin_1)
- net SCLK: now also J3.23 (BCM11)
- net at J2.1, R5.1: now also U2.7 (WP)
- net TC+: no longer names the net of C3.1, J1.2 (Pin_2), U1.4 (T+)
- net TC+: now also C1.1; no longer C1.2
- net TC-: no longer names the net of C3.2, J1.1 (Pin_1), U1.2 (BIAS), U1.3 (T-)
- net TC-: now also C2.2; no longer C2.1
- net TC_CS renamed ~TC_CS
- net ~TC_CS: now also J3.33 (BCM13)
- net TC_FAULT renamed ~TC_FAULT
- net ~TC_FAULT: now also J3.35 (BCM19)
- net TC_~DRDY renamed ~TC_DRDY
- net ~TC_DRDY: now also J3.37 (BCM26)
- new net: D1.2 (A), R1.1
- new net: J4.2 (Pin_2), R1.2
- new net: J4.10 (Pin_10), R8.2
- new net: J4.12 (Pin_12), R9.2
- new net: J4.4 (Pin_4), R2.2
- new net: J4.6 (Pin_6), R3.2
- new net: J4.8 (Pin_8), R4.2
- new net: D2.2 (A), R2.1
- new net: D3.2 (A), R3.1
- new net: D4.2 (A), R4.1
- new net: D5.2 (A), R8.1
- new net: D6.2 (A), R9.1
- new net 3V3_MAX: C4.2, C5.2, J4.5 (Pin_5), R10.1, U1.5 (AVDD), U1.8 (DVDD), U3.3
- new net SOUND: J3.40 (BCM21), R?.2
- new net TC_RESET: J3.7 (BCM4), U3.1
- no-connect marks 18 -> 12
Other:
- note added: "TC POWER-CYCLE RELAY"
- note added: "TODO: add sound switch to turn off sound logic"
- note added: "TODO: correct poinout for easiest routing"
- note added: "TODO: toggle switch for sound"
- note added: "pd resistor to drain tc chip caps on reset"
- note removed: "TEST POINTS"
- note removed: "THERMOCOUPLE CONNECTOR"
- moved on the sheet: C1, C2, C3, C4, C5, C6, J1, J2, R5, R6, R7, U1

Commit message: continued layout, some routing & pinout changes
Parts:
- H1, H2, H3, H4: footprint project_footprints:NPTH_3mm_ID -> MountingHole:MountingHole_2.7mm_M2.5_DIN965
- R11: renamed from R?; footprint (none) -> Connector_PinHeader_2.54mm:PinHeader_2x01_P2.54mm_Vertical
Connections:
- net +3V3: now also J4.7 (Pin_7); no longer J4.11 (Pin_11)
- net FAULT: now also J4.1 (Pin_1); no longer J4.7 (Pin_7)
- net HBEAT: now also J4.3 (Pin_3); no longer J3.38 (BCM20), J4.9 (Pin_9)
- net MISO: now also J4.9 (Pin_9); no longer J4.3 (Pin_3)
- net MOSI: now also J4.11 (Pin_11); no longer J4.1 (Pin_1)
- net SOUND: now also J3.11 (BCM17); no longer J3.40 (BCM21)
- net TC_RESET: now also J3.10 (BCM15); no longer J3.7 (BCM4)
- net ~TC_CS: now also J3.38 (BCM20); no longer J3.33 (BCM13)
- net ~TC_DRDY: now also J3.40 (BCM21); no longer J3.37 (BCM26)
- net ~TC_FAULT: now also J3.8 (BCM14); no longer J3.35 (BCM19)
- net TC+: now reaches C1.1, C3.1, J1.2 (Pin_2), U1.4 (T+)
- net TC-: now reaches C2.2, C3.2, J1.1 (Pin_1), U1.2 (BIAS), U1.3 (T-)
- no-connect marks 12 -> 7
Changed lines of the file:
@@
 	7700 5650 7750 5650
 Wire Wire Line
+	9900 6350 9850 6350
+Wire Wire Line
+	9000 6350 8950 6350
+Wire Wire Line
 	9000 6450 8950 6450
 Wire Wire Line
-	9000 6350 8950 6350
-Wire Wire Line
-	7700 6250 7750 6250
-Wire Wire Line
-	7750 6350 7700 6350
+	8950 4950 9000 4950
 Text Notes 13300 3600 0    118  ~ 24
 THERMOCOUPLE
@@
 Wire Wire Line
 	12700 2150 12700 2200
-Text Label 9000 6450 0    50   ~ 0
+Text Label 9900 6350 0    50   ~ 0
 HBEAT
 Text Label 9000 6350 0    50   ~ 0
 FAULT
-Text Label 7700 6250 2    50   ~ 0
+Text Label 9000 6450 0    50   ~ 0
 ~TC_CS
-Text Label 7700 6350 2    50   ~ 0
-~TC_FAULT
-Text Label 7700 6450 2    50   ~ 0
+Text Label 9000 6550 0    50   ~ 0
 ~TC_DRDY
 Text Label 9000 5950 0    50   ~ 0
@@
 Wire Wire Line
 	7000 6550 7000 6600
-NoConn ~ 8950 4950
-NoConn ~ 8950 5050
 NoConn ~ 8950 5150
 Wire Wire Line
@@
 NoConn ~ 7750 6150
 NoConn ~ 7750 5250
-NoConn ~ 7750 5150
 $Comp
 L power:PWR_FLAG #FLG03
@@
 Wire Wire Line
 	14500 8900 14500 9000
-Text Label 1900 4000 2    50   ~ 0
-FAULT
-Text Label 1900 4100 2    50   ~ 0
-HBEAT
 $Comp
 L Connector_Generic:Conn_02x06_Odd_Even J4
@@
 F 0 "H1" H 1800 9746 50  0000 L CNN
 F 1 "MountingHole" H 1800 9655 50  0000 L CNN
-F 2 "project_footprints:NPTH_3mm_ID" H 1700 9700 50  0001 C CNN
+F 2 "MountingHole:MountingHole_2.7mm_M2.5_DIN965" H 1700 9700 50  0001 C CNN
 F 3 "~" H 1700 9700 50  0001 C CNN
 	1    1700 9700
@@
 F 0 "H2" H 1800 9946 50  0000 L CNN
 F 1 "MountingHole" H 1800 9855 50  0000 L CNN
-F 2 "project_footprints:NPTH_3mm_ID" H 1700 9900 50  0001 C CNN
+F 2 "MountingHole:MountingHole_2.7mm_M2.5_DIN965" H 1700 9900 50  0001 C CNN
 F 3 "~" H 1700 9900 50  0001 C CNN
 	1    1700 9900
@@
 F 0 "H3" H 1800 10146 50  0000 L CNN
 F 1 "MountingHole" H 1800 10055 50  0000 L CNN
-F 2 "project_footprints:NPTH_3mm_ID" H 1700 10100 50  0001 C CNN
+F 2 "MountingHole:MountingHole_2.7mm_M2.5_DIN965" H 1700 10100 50  0001 C CNN
 F 3 "~" H 1700 10100 50  0001 C CNN
 	1    1700 10100
@@
 F 0 "H4" H 1800 10346 50  0000 L CNN
 F 1 "MountingHole" H 1800 10255 50  0000 L CNN
-F 2 "project_footprints:NPTH_3mm_ID" H 1700 10300 50  0001 C CNN
+F 2 "MountingHole:MountingHole_2.7mm_M2.5_DIN965" H 1700 10300 50  0001 C CNN
 F 3 "~" H 1700 10300 50  0001 C CNN
 	1    1700 10300
@@
 $EndComp
 Wire Wire Line
-	7750 6450 7700 6450
+	8950 6550 9000 6550
 NoConn ~ 8950 5850
 Wire Wire Line
@@
 Text Notes 2150 6350 0    50   ~ 0
 TODO: add sound switch to turn off sound logic
-Text Label 7700 4950 2    50   ~ 0
+Text Label 9000 5050 0    50   ~ 0
 TC_RESET
 Wire Wire Line
-	7700 4950 7750 4950
-Wire Wire Line
-	1900 4000 2000 4000
-Wire Wire Line
-	1900 4100 2000 4100
+	9000 5050 8950 5050
 $Comp
 L power:+3V3 #PWR0103
 U 1 1 61762891
-P 1400 4100
-F 0 "#PWR0103" H 1400 3950 50  0001 C CNN
-F 1 "+3V3" H 1415 4273 50  0000 C CNN
-F 2 "" H 1400 4100 50  0001 C CNN
-F 3 "" H 1400 4100 50  0001 C CNN
-	1    1400 4100
-	1    0    0    -1
-$EndComp
-Wire Wire Line
-	1400 4100 1400 4200
+P 1400 3900
+F 0 "#PWR0103" H 1400 3750 50  0001 C CNN
+F 1 "+3V3" H 1415 4073 50  0000 C CNN
+F 2 "" H 1400 3900 50  0001 C CNN
+F 3 "" H 1400 3900 50  0001 C CNN
+	1    1400 3900
+	1    0    0    -1
+$EndComp
+Wire Wire Line
+	1400 3900 1400 4000
 Text Label 1900 3900 2    50   ~ 0
 3V3_MAX
@@
 	1900 3900 2000 3900
 Wire Wire Line
-	1400 4200 2000 4200
-Text Label 1900 3700 2    50   ~ 0
+	1400 4000 2000 4000
+Text Label 1900 4200 2    50   ~ 0
 MOSI
-Text Label 1900 3800 2    50   ~ 0
+Text Label 1900 4100 2    50   ~ 0
 MISO
 Wire Wire Line
-	1900 3800 2000 3800
-Wire Wire Line
-	2000 3700 1900 3700
+	1900 4100 2000 4100
+Wire Wire Line
+	2000 4200 1900 4200
+NoConn ~ 7750 6050
+NoConn ~ 7750 5350
+$Comp
+L Device:R R11
+U 1 1 6181A47C
+P 8200 8900
+F 0 "R11" V 7993 8900 50  0000 C CNN
+F 1 "R" V 8084 8900 50  0000 C CNN
+F 2 "Connector_PinHeader_2.54mm:PinHeader_2x01_P2.54mm_Vertical" V 8130 8900 50  0001 C CNN
+F 3 "~" H 8200 8900 50  0001 C CNN
+	1    8200 8900
+	0    1    1    0
+$EndComp
+Text Label 7950 8900 2    50   ~ 0
+SOUND
+Wire Wire Line
+	7950 8900 8050 8900
+Wire Wire Line
+	8350 8900 8550 8900
+$Comp
+L power:GND #PWR01
+U 1 1 6182C40F
+P 8550 8900
+F 0 "#PWR01" H 8550 8650 50  0001 C CNN
+F 1 "GND" H 8555 8727 50  0000 C CNN
+F 2 "" H 8550 8900 50  0001 C CNN
+F 3 "" H 8550 8900 50  0001 C CNN
+	1    8550 8900
+	1    0    0    -1
+$EndComp
+Text Notes 7750 9300 0    50   ~ 0
+TODO: toggle switch for sound
+Text Label 7700 5150 2    50   ~ 0
+SOUND
+Wire Wire Line
+	7700 5150 7750 5150
 $Comp
 L calciHATter:PI40HAT J3
@@
 	1    0    0    -1
 $EndComp
-NoConn ~ 7750 6050
-NoConn ~ 7750 5350
-$Comp
-L Device:R R?
-U 1 1 6181A47C
-P 8200 8900
-F 0 "R?" V 7993 8900 50  0000 C CNN
-F 1 "R" V 8084 8900 50  0000 C CNN
-F 2 "" V 8130 8900 50  0001 C CNN
-F 3 "~" H 8200 8900 50  0001 C CNN
-	1    8200 8900
-	0    1    1    0
-$EndComp
-Text Label 7950 8900 2    50   ~ 0
-SOUND
-Wire Wire Line
-	7950 8900 8050 8900
-Wire Wire Line
-	8350 8900 8550 8900
-$Comp
-L power:GND #PWR?
-U 1 1 6182C40F
-P 8550 8900
-F 0 "#PWR?" H 8550 8650 50  0001 C CNN
-F 1 "GND" H 8555 8727 50  0000 C CNN
-F 2 "" H 8550 8900 50  0001 C CNN
-F 3 "" H 8550 8900 50  0001 C CNN
-	1    8550 8900
-	1    0    0    -1
-$EndComp
-Text Notes 7750 9300 0    50   ~ 0
-TODO: toggle switch for sound
-Text Label 9000 6550 0    50   ~ 0
-SOUND
-Wire Wire Line
-	9000 6550 8950 6550
-NoConn ~ 7750 4750
-NoConn ~ 7750 4850
+Text Label 9000 4950 0    50   ~ 0
+~TC_FAULT
+Wire Wire Line
+	1900 3800 2000 3800
+Wire Wire Line
+	1900 3700 2000 3700
+Text Label 1900 3800 2    50   ~ 0
+HBEAT
+Text Label 1900 3700 2    50   ~ 0
+FAULT
+Text Label 13500 4600 2    50   ~ 0
+TC+
+Text Label 13500 4900 2    50   ~ 0
+TC-
 $EndSCHEMATC

Commit message: Finalized pinout, routing. TODO: cleanup+ERC
Parts:
- removed R11: R, Connector_PinHeader_2.54mm:PinHeader_2x01_P2.54mm_Vertical, symbol Device:R
- added R11, R12: 100, Resistor_SMD:R_0603_1608Metric_Pad1.05x0.95mm_HandSolder, symbol Device:R_Small
- added SW1: SW_SPDT, Connector_PinHeader_2.54mm:PinHeader_1x03_P2.54mm_Vertical, symbol Switch:SW_SPDT
- C4, C5: value 100n -> 100n, 0603
- D1: value GREEN, 0603 -> RED
- D2: value RED, 0603 -> AMBER
- D3, D4: value GREEN, 0603 -> GREEN
- D5, D6: value GREEN, 0603 -> AMBER
- R1, R2, R3, R4, R8, R9: value 1k, 0603 -> 1k
- R10: value 10k, 0603, 1% -> 10k
Connections:
- net +3V3: now also J4.11 (Pin_11); no longer J4.7 (Pin_7)
- net FAULT: now also J3.7 (BCM4), J4.7 (Pin_7); no longer J3.36 (BCM16), J4.1 (Pin_1)
- net GND: now also SW1.3 (C)
- net HBEAT: now also J3.13 (BCM27), J4.9 (Pin_9); no longer J4.3 (Pin_3)
- net MISO: now also J4.3 (Pin_3); no longer J4.9 (Pin_9)
- net MOSI: now also J4.1 (Pin_1); no longer J4.11 (Pin_11)
- net SOUND: now also J3.3 (BCM2), SW1.2 (B); no longer J3.11 (BCM17)
- net TC+: now also R11.2; no longer C1.1, C3.1, U1.4 (T+)
- net TC-: now also R12.2; no longer C2.2, C3.2, U1.3 (T-)
- net TC_RESET: now also J3.5 (BCM3); no longer J3.10 (BCM15)
- net ~TC_FAULT: now also J3.11 (BCM17); no longer J3.8 (BCM14)
- new net: C1.1, C3.1, R11.1, U1.4 (T+)
- new net: C2.2, C3.2, R12.1, U1.3 (T-)
Other:
- note added: "\nhttps://cdn-learn.adafruit.com/assets/assets/000/035/946/original/sensors_schem.png?1474583748"
- note removed: "TODO: toggle switch for sound"
- moved on the sheet: C1, C2, C3, C4, C5, C6, H1, H2, H3, H4, J1, J2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

Commit message: finalized schematic+routing. need easter eggs and footprint checks
Connections:
- net +5C: no longer names the net of J3.2 (P5V)
- net +5C: no longer J3.4 (P5V)
- no-connect marks 7 -> 19
Other:
- note added: "- Use RPi internal pull up on sound switch"
- note added: "FIRMWARE NOTES"
- note added: "SOUND CONTROL SWITCH"
- note removed: "TODO: add sound switch to turn off sound logic"
- moved on the sheet: C1, C2, C3, C4, C5, C6, D1, D2, D3, D4, D5, D6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
